File: preamp2.kicad_pcb (KiCad board)
At the start: 2 copper layers, 32 x 4 mm, 12 parts, among them J1 piezo, J2 output, U1 OPA1677

Commit message: A few more tweaks in components, after more measurements.
Other:
- board text added: "GND"
- board text added: "INPUT"
- board text added: "OUTPUT"
- board text added: "VCC"
Changed lines of the file:
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@@
     (fp_line (start 1 5) (end -1 5)
       (stroke (width 0.1) (type solid)) (layer "F.Fab"))
-    (pad "1" thru_hole rect (at 0 0 90) (size 1.35 1.35) (drill 0.6) (layers "*.Cu" "*.Mask")
+    (pad "1" thru_hole rect (at 0 0 90) (size 1.35 1.35) (drill 0.8) (layers "*.Cu" "*.Mask")
       (net 7 "+9V") (pinfunction "Pin_1") (pintype "passive"))
-    (pad "2" thru_hole oval (at 0 2 90) (size 1.35 1.35) (drill 0.6) (layers "*.Cu" "*.Mask")
+    (pad "2" thru_hole oval (at 0 2 90) (size 1.35 1.35) (drill 0.8) (layers "*.Cu" "*.Mask")
       (net 5 "Net-(J2-Pin_2)") (pinfunction "Pin_2") (pintype "passive"))
-    (pad "3" thru_hole oval (at 0 4 90) (size 1.35 1.35) (drill 0.6) (layers "*.Cu" "*.Mask")
+    (pad "3" thru_hole oval (at 0 4 90) (size 1.35 1.35) (drill 0.8) (layers "*.Cu" "*.Mask")
       (net 1 "GND") (pinfunction "Pin_3") (pintype "passive"))
     (model "${KICAD6_3DMODEL_DIR}/Connector_PinHeader_2.00mm.3dshapes/PinHeader_1x03_P2.00mm_Vertical.wrl"
@@
   (gr_line (start 125.5 90) (end 125.5 94)
     (stroke (width 0.1) (type default)) (layer "Edge.Cuts"))
+  (gr_text "VCC" (at 119.888 89.662 90) (layer "Dwgs.User")
+    (effects (font (size 0.65 0.65) (thickness 0.1)) (justify left bottom))
+  )
+  (gr_text "OUTPUT" (at 121.666 89.662 90) (layer "Dwgs.User")
+    (effects (font (size 0.65 0.65) (thickness 0.1)) (justify left bottom))
+  )
+  (gr_text "GND" (at 95.758 89.662 90) (layer "Dwgs.User")
+    (effects (font (size 0.65 0.65) (thickness 0.1)) (justify left bottom))
+  )
+  (gr_text "INPUT" (at 97.79 89.662 90) (layer "Dwgs.User")
+    (effects (font (size 0.65 0.65) (thickness 0.1)) (justify left bottom))
+  )
+  (gr_text "GND" (at 123.698 89.662 90) (layer "Dwgs.User")
+    (effects (font (size 0.65 0.65) (thickness 0.1)) (justify left bottom))
+  )
   (dimension (type aligned) (layer "B.Cu")
     (pts (xy 93.5 94) (xy 125.5 94))
