File: preamp2.kicad_sch (KiCad schematic)
At the start: 18 parts, among them J1 piezo, J2 output, J3 piezo, J4 Conn_01x03_Pin, J5 AudioJack3, U1 OPA1677

Commit message: Tweaked some component values.
Parts:
- C1: value 1u -> 220n
- C4: value 1u -> 2u2
- J5: value AudioJack3 -> AudioJack
Changed lines of the file:
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@@
       (effects (font (size 1.27 1.27)) (justify left))
     )
-    (property "Value" "1u" (at 93.98 92.075 0)
+    (property "Value" "220n" (at 92.71 92.075 0)
       (effects (font (size 1.27 1.27)) (justify left))
     )
@@
       (effects (font (size 1.27 1.27)) (justify left))
     )
-    (property "Value" "1u" (at 140.335 75.565 0)
+    (property "Value" "2u2" (at 140.335 75.565 0)
       (effects (font (size 1.27 1.27)) (justify left))
     )
@@
   (symbol (lib_id "Connector_Audio:AudioJack3") (at 188.595 88.265 180) (unit 1)
     (in_bom yes) (on_board yes) (dnp no) (fields_autoplaced)
-    (property "Reference" "J5" (at 196.85 86.995 0)
+    (property "Reference" "J5" (at 196.85 86.36 0)
       (effects (font (size 1.27 1.27)) (justify right))
     )
-    (property "Value" "AudioJack3" (at 196.85 89.535 0)
+    (property "Value" "AudioJack" (at 196.85 88.9 0)
       (effects (font (size 1.27 1.27)) (justify right))
     )

Commit message: Tweaked some component values, again.
Parts:
- R3, R4: value 820k -> 1M
Changed lines of the file:
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@@
   )
   (symbol (lib_id "Device:R") (at 90.17 83.185 90) (unit 1)
-    (in_bom yes) (on_board yes) (dnp no) (fields_autoplaced)
-    (property "Reference" "R3" (at 90.17 78.74 90)
-      (effects (font (size 1.27 1.27)))
-    )
-    (property "Value" "820k" (at 90.17 81.28 90)
+    (in_bom yes) (on_board yes) (dnp no)
+    (property "Reference" "R3" (at 90.17 79.375 90)
+      (effects (font (size 1.27 1.27)))
+    )
+    (property "Value" "1M" (at 90.17 81.28 90)
       (effects (font (size 1.27 1.27)))
     )
@@
   (symbol (lib_id "Device:D_TVS") (at 83.185 90.17 90) (unit 1)
     (in_bom yes) (on_board yes) (dnp no)
-    (property "Reference" "D1" (at 85.09 88.9 90)
-      (effects (font (size 1.27 1.27)) (justify right))
-    )
-    (property "Value" "TVS 6V" (at 85.09 92.075 90)
+    (property "Reference" "D1" (at 78.74 88.265 90)
+      (effects (font (size 1.27 1.27)) (justify right))
+    )
+    (property "Value" "TVS 6V" (at 85.09 88.265 90)
       (effects (font (size 1.27 1.27)) (justify right))
     )
@@
   )
   (symbol (lib_id "Device:R") (at 121.285 88.9 90) (unit 1)
-    (in_bom yes) (on_board yes) (dnp no) (fields_autoplaced)
-    (property "Reference" "R4" (at 121.285 84.455 90)
-      (effects (font (size 1.27 1.27)))
-    )
-    (property "Value" "820k" (at 121.285 86.995 90)
-      (effects (font (size 1.27 1.27)))
-    )
+    (in_bom yes) (on_board yes) (dnp no)
+    (property "Reference" "R4" (at 121.285 85.09 90)
+      (effects (font (size 1.27 1.27)))
+    )
+    (property "Value" "1M" (at 121.285 86.995 90)
+      (effects (font (size 1.27 1.27)))
+    )

Commit message: A few more tweaks in components, after more measurements.
Parts:
- C2: value 10p -> 39p
- D1: value TVS 6V -> TVS 2V5
Changed lines of the file:
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@@
       (effects (font (size 1.27 1.27)))
     )
-    (property "Value" "10p" (at 125.095 95.25 90)
+    (property "Value" "39p" (at 125.095 95.25 90)
       (effects (font (size 1.27 1.27)))
     )
@@
       (effects (font (size 1.27 1.27)) (justify right))
     )
-    (property "Value" "TVS 6V" (at 85.09 88.265 90)
+    (property "Value" "TVS 2V5" (at 86.614 86.106 0)
       (effects (font (size 1.27 1.27)) (justify right))
     )
